Commit message: refactor: Change my robot model

File: src/my_robot/urdf/my_robot.xacro (robot description, xacro)
@@ -1,310 +1,188 @@
-<?xml version='1.0'?>
+<?xml version="1.0"?>
 <robot name="my_robot" xmlns:xacro="http://www.ros.org/wiki/xacro">
+  <xacro:include filename="$(find my_robot)/urdf/my_robot.gazebo" />
   <link name="robot_footprint"></link>
-  <xacro:include filename="$(find my_robot)/urdf/my_robot.gazebo"/>
   <joint name="robot_footprint_joint" type="fixed">
-    <origin xyz="0 0 0" rpy="0 0 0"/>
-    <parent link="robot_footprint"/>
-    <child link="chassis"/>
+    <origin xyz="0 0 0" rpy="0 0 0" />
+    <parent link="robot_footprint" />
+    <child link="chassis" />
   </joint>
-  <link name='chassis'>
+  <link name="chassis">
     <pose>0 0 0.1 0 0 0</pose>
     <inertial>
-      <mass value="10.0"/>
-      <origin xyz="0.0 0 0" rpy=" 0 0 0"/>
+      <mass value="15.0" />
+      <origin xyz="0 0 0" rpy="0 0 0" />
       <inertia
-          ixx="0.1" ixy="0" ixz="0"
-          iyy="0.1" iyz="0"
-          izz="0.1"
+        ixx="0.1" ixy="0" ixz="0"
+        iyy="0.1" iyz="0"
+        izz="0.1"
       />
     </inertial>
-    <collision name='chassis_collision'>
-      <origin xyz="0 0 0" rpy=" 0 0 0"/>
+    <collision name="chassis_collision_1">
+      <origin xyz="-.2 0 0" rpy="0 0 0" />
       <geometry>
-        <box size="2. .9 .1"/>
+        <box size="1.0 .2 .1" />
       </geometry>
     </collision>
-    <visual name='chassis_visual'>
-      <origin xyz="0 0 0" rpy=" 0 0 0"/>
+    <visual name="chassis_visual_1">
+      <origin xyz="-.2 0 0" rpy="0 0 0" />
       <geometry>
-        <box size="2. .9 .1"/>
+        <box size="1.0 .2 .1" />
       </geometry>
     </visual>
-    <collision name='sensor_platform_collision'>
-      <origin xyz="0.8 0 0.1" rpy=" 0 0 0"/>
+    <collision name="chassis_collision_2">
+      <origin xyz="0 0 0" rpy="0 0 0" />
       <geometry>
-        <box size=".1 .1 .3"/>
+        <box size=".2 .6 .1" />
       </geometry>
     </collision>
-    <visual name='sensor_platform_visual'>
-      <origin xyz="0.8 0 0.1" rpy=" 0 0 0"/>
+    <visual name="chassis_visual_2">
+      <origin xyz="0 0 0" rpy="0 0 0" />
       <geometry>
-        <box size=".1 .1 .3"/>
+        <box size=".2 .6 .1" />
       </geometry>
     </visual>
-    <collision name='front_left_caster_collision'>
-      <origin xyz="0.9 .35 -0.05" rpy=" 0 0 0"/>
+    <collision name="back_caster_collision">
+      <origin xyz="-0.65 0 -0.05" rpy="0 0 0" />
       <geometry>
-        <sphere radius="0.0499"/>
+        <sphere radius="0.0499" />
       </geometry>
     </collision>
-    <visual name='front_left_caster_visual'>
-      <origin xyz="0.9 .35 -0.05" rpy=" 0 0 0"/>
+    <visual name="back_caster_visual">
+      <origin xyz="-0.65 0 -0.05" rpy="0 0 0" />
       <geometry>
-        <sphere radius="0.05"/>
+        <sphere radius="0.0499" />
       </geometry>
     </visual>
-    <collision name='front_right_caster_collision'>
-      <origin xyz="0.9 -0.35 -0.05" rpy=" 0 0 0"/>
+    <collision name="front_caster_collision">
+      <origin xyz="0.25 0 -0.05" rpy="0 0 0" />
       <geometry>
-        <sphere radius="0.0499"/>
+        <sphere radius="0.0499" />
       </geometry>
     </collision>
-    <visual name='front_right_caster_visual'>
-      <origin xyz="0.9 -0.35 -0.05" rpy=" 0 0 0"/>
+    <visual name="front_caster_visual">
+      <origin xyz="0.25 0 -0.05" rpy="0 0 0" />
       <geometry>
-        <sphere radius="0.05"/>
-      </geometry>
-    </visual>
-    <collision name='center_left_caster_collision'>
-      <origin xyz="0 0.35 -0.05" rpy=" 0 0 0"/>
-      <geometry>
-        <sphere radius="0.0499"/>
-      </geometry>
-    </collision>
-    <visual name='center_left_caster_visual'>
-      <origin xyz="0 0.35 -0.05" rpy=" 0 0 0"/>
-      <geometry>
-        <sphere radius="0.05"/>
-      </geometry>
-    </visual>
-    <collision name='center_right_caster_collision'>
-      <origin xyz="0 -0.35 -0.05" rpy=" 0 0 0"/>
-      <geometry>
-        <sphere radius="0.0499"/>
-      </geometry>
-    </collision>
-    <visual name='center_right_caster_visual'>
-      <origin xyz="0 -0.35 -0.05" rpy=" 0 0 0"/>
-      <geometry>
-        <sphere radius="0.05"/>
-      </geometry>
-    </visual>
-    <collision name='rear_left_caster_collision'>
-      <origin xyz="-0.9 0.35 -0.05" rpy=" 0 0 0"/>
-      <geometry>
-        <sphere radius="0.0499"/>
-      </geometry>
-    </collision>
-    <visual name='rear_left_caster_visual'>
-      <origin xyz="-0.9 0.35 -0.05" rpy=" 0 0 0"/>
-      <geometry>
-        <sphere radius="0.05"/>
-      </geometry>
-    </visual>
-    <collision name='rear_right_caster_collision'>
-      <origin xyz="-0.9 -0.35 -0.05" rpy=" 0 0 0"/>
-      <geometry>
-        <sphere radius="0.0499"/>
-      </geometry>
-    </collision>
-    <visual name='rear_right_caster_visual'>
-      <origin xyz="-0.9 -0.35 -0.05" rpy=" 0 0 0"/>
-      <geometry>
-        <sphere radius="0.05"/>
+        <sphere radius="0.0499" />
       </geometry>
     </visual>
   </link>
-  <link name='front_left_wheel'>
-    <pose>0 0 0 0 0 0</pose>
+  <link name="left_wheel">
     <inertial>
-      <mass value="5.0"/>
-      <origin xyz="0.0 0 0" rpy=" 0 1.5707 1.5707"/>
+      <mass value="5.0" />
+      <origin xyz="0 0 0" rpy="0 1.5707 1.5707" />
       <inertia
-          ixx="0.1" ixy="0" ixz="0"
-          iyy="0.1" iyz="0"
-          izz="0.1"
+        ixx="0.1" ixy="0" ixz="0"
+        iyy="0.1" iyz="0"
+        izz="0.1"
       />
     </inertial>
-    <collision name='front_left_wheel_collision'>
-      <origin xyz="0 0 0" rpy=" 0 1.5707 1.5707"/>
+    <collision>
+      <origin xyz="0 0 0" rpy="0 1.5707 1.5707" />
       <geometry>
-        <cylinder radius="0.14" length="0.21"/>
+        <cylinder radius="0.1" length="0.05" />
       </geometry>
     </collision>
-    <visual name='front_left_wheel_visual'>
-      <origin xyz="0 0 0" rpy=" 0 1.5707 1.5707"/>
+    <visual>
+      <origin xyz="0 0 0" rpy="0 1.5707 1.5707" />
       <geometry>
-        <cylinder radius="0.14" length="0.21"/>
+        <cylinder radius="0.1" length="0.05" />
       </geometry>
     </visual>
   </link>
-  <link name='front_right_wheel'>
-    <pose>0 0 0 0 0 0</pose>
+  <link name="right_wheel">
     <inertial>
-      <mass value="5.0"/>
-      <origin xyz="0.0 0 0" rpy=" 0 1.5707 1.5707"/>
+      <mass value="5.0" />
+      <origin xyz="0 0 0" rpy="0 1.5707 1.5707" />
       <inertia
-          ixx="0.1" ixy="0" ixz="0"
-          iyy="0.1" iyz="0"
-          izz="0.1"
+        ixx="0.1" ixy="0" ixz="0"
+        iyy="0.1" iyz="0"
+        izz="0.1"
       />
     </inertial>
-    <collision name='front_right_wheel_collision'>
-      <origin xyz="0 0 0" rpy=" 0 1.5707 1.5707"/>
+    <collision>
+      <origin xyz="0 0 0" rpy="0 1.5707 1.5707" />
       <geometry>
-        <cylinder radius="0.14" length="0.21"/>
+        <cylinder radius="0.1" length="0.05" />
       </geometry>
     </collision>
-    <visual name='front_right_wheel_visual'>
-      <origin xyz="0 0 0" rpy=" 0 1.5707 1.5707"/>
+    <visual>
+      <origin xyz="0 0 0" rpy="0 1.5707 1.5707" />
       <geometry>
-        <cylinder radius="0.14" length="0.21"/>
+        <cylinder radius="0.1" length="0.05" />
       </geometry>
     </visual>
   </link>
-  <link name='rear_left_wheel'>
-    <pose>0 0 0 0 0 0</pose>
-    <inertial>
-      <mass value="5.0"/>
-      <origin xyz="0.0 0 0" rpy=" 0 1.5707 1.5707"/>
-      <inertia
-          ixx="0.1" ixy="0" ixz="0"
-          iyy="0.1" iyz="0"
-          izz="0.1"
-      />
-    </inertial>
-    <collision name='rear_left_wheel_collision'>
-      <origin xyz="0 0 0" rpy=" 0 1.5707 1.5707"/>
+  <gazebo reference="left_wheel">
+    <material>Gazebo/Blue</material>
+  </gazebo>
+  <gazebo reference="right_wheel">
+    <material>Gazebo/Red</material>
+  </gazebo>
+  <joint type="continuous" name="left_wheel_hinge">
+    <origin xyz="0 0.325 0" rpy="0 0 0" />
+    <child link="left_wheel" />
+    <parent link="chassis" />
+    <axis xyz="0 1 0" rpy="0 0 0" />
+    <limit effort="10000" velocity="1000" />
+    <dynamics damping="1.0" friction="1.0" />
+  </joint>
+  <joint type="continuous" name="right_wheel_hinge">
+    <origin xyz="0 -0.325 0" rpy="0 0 0" />
+    <child link="right_wheel" />
+    <parent link="chassis" />
+    <axis xyz="0 1 0" rpy="0 0 0" />
+    <limit effort="10000" velocity="1000" />
+    <dynamics damping="1.0" friction="1.0" />
+  </joint>
+  <link name="camera">
+    <box_inertia x="0.05" y="0.05" z="0.05" m="0.1" />
+    <collision>
+      <origin xyz="0 0 0" rpy="0 0 0" />
       <geometry>
-        <cylinder radius="0.14" length="0.21"/>
+        <box size="0.05 0.05 0.05" />
       </geometry>
     </collision>
-    <visual name='rear_left_wheel_visual'>
-      <origin xyz="0 0 0" rpy=" 0 1.5707 1.5707"/>
+    <visual>
+      <origin xyz="0 0 0" rpy="0 0 0" />
       <geometry>
-        <cylinder radius="0.14" length="0.21"/>
+        <box size="0.05 0.05 0.05" />
       </geometry>
     </visual>
   </link>
-  <link name='rear_right_wheel'>
-    <pose>0 0 0 0 0 0</pose>
+  <gazebo reference="camera">
+    <material>Gazebo/Green</material>
+  </gazebo>
+  <joint type="fixed" name="camera_joint">
+    <origin xyz="0.3 0 0" rpy="0 0 0" />
+    <parent link="chassis" />
+    <child link="camera" />
+  </joint>
+  <link name="hokuyo">
     <inertial>
-      <mass value="5.0"/>
-      <origin xyz="0.0 0 0" rpy=" 0 1.5707 1.5707"/>
+      <mass value="1e-5" />
       <inertia
-          ixx="0.1" ixy="0" ixz="0"
-          iyy="0.1" iyz="0"
-          izz="0.1"
+        ixx="1e-6" ixy="0" ixz="0"
+        iyy="1e-6" iyz="0"
+        izz="1e-6"
       />
     </inertial>
-    <collision name='rear_right_wheel_collision'>
-      <origin xyz="0 0 0" rpy=" 0 1.5707 1.5707"/>
+    <collision>
+      <origin xyz="0 0 0" rpy="0 0 0" />
       <geometry>
-        <cylinder radius="0.14" length="0.21"/>
+        <box size="0.1 0.1 0.1" />
       </geometry>
     </collision>
-    <visual name='rear_right_wheel_visual'>
-      <origin xyz="0 0 0" rpy=" 0 1.5707 1.5707"/>
+    <visual>
+      <origin xyz="0 0 0" rpy="0 0 0" />
       <geometry>
-        <cylinder radius="0.14" length="0.21"/>
+        <mesh filename="package://my_robot/meshes/hokuyo.dae" />
       </geometry>
     </visual>
   </link>
-  <joint type="continuous" name="front_left_wheel_hinge">
-    <origin xyz="0.9 0.6 0" rpy="0 0 0"/>
-    <child link="front_left_wheel"/>
-    <parent link="chassis"/>
-    <axis xyz="0 1 0" rpy="0 0 0"/>
-    <limit effort="10000" velocity="1000"/>
-    <dynamics damping="1.0" friction="1.0"/>
-  </joint>
-  <joint type="continuous" name="front_right_wheel_hinge">
-    <origin xyz="0.9 -0.6 0" rpy="0 0 0"/>
-    <child link="front_right_wheel"/>
-    <parent link="chassis"/>
-    <axis xyz="0 1 0" rpy="0 0 0"/>
-    <limit effort="10000" velocity="1000"/>
-    <dynamics damping="1.0" friction="1.0"/>
-  </joint>
-  <joint type="continuous" name="rear_left_wheel_hinge">
-    <origin xyz="-0.9 0.6 0" rpy="0 0 0"/>
-    <child link="rear_left_wheel"/>
-    <parent link="chassis"/>
-    <axis xyz="0 1 0" rpy="0 0 0"/>
-    <limit effort="10000" velocity="1000"/>
-    <dynamics damping="1.0" friction="1.0"/>
-  </joint>
-  <joint type="continuous" name="rear_right_wheel_hinge">
-    <origin xyz="-0.9 -0.6 0" rpy="0 0 0"/>
-    <child link="rear_right_wheel"/>
-    <parent link="chassis"/>
-    <axis xyz="0 1 0" rpy="0 0 0"/>
-    <limit effort="10000" velocity="1000"/>
-    <dynamics damping="1.0" friction="1.0"/>
-  </joint>
-  <link name='camera'>
-    <pose>0 0 0 0 0 0</pose>
-    <inertial>
-      <mass value="0.1"/>
-      <origin xyz="0.0 0 0" rpy="0.0 0 0"/>
-      <inertia
-          ixx="1e-6" ixy="0" ixz="0"
-          iyy="1e-6" iyz="0"
-          izz="1e-6"
-      />
-    </inertial>
-    <collision name='collision'>
-      <origin xyz="0 0 0" rpy=" 0 0 0"/>
-      <geometry>
-        <box size="0.05 0.05 0.05"/>
-      </geometry>
-    </collision>
-    <visual name='camera_visual'>
-      <origin xyz="0 0 0" rpy="0 0 0"/>
-      <geometry>
-        <box size="0.05 0.05 0.05"/>
-      </geometry>
-    </visual>
-  </link>
-  <joint type="fixed" name="camera_joint">
-    <origin xyz="1.0 0 0" rpy="0 0 0"/>
-    <child link="camera"/>
-    <parent link="chassis"/>
-    <axis xyz="0 1 0" rpy="0 0 0"/>
-    <limit effort="10000" velocity="1000"/>
-    <dynamics damping="1.0" friction="1.0"/>
-  </joint>
-  <link name='hokuyo'>
-    <pose>0 0 0 0 0 0</pose>
-    <inertial>
-      <mass value="1e-5"/>
-      <origin xyz="0.0 0 0" rpy="0.0 0 0"/>
-      <inertia
-          ixx="1e-6" ixy="0" ixz="0"
-          iyy="1e-6" iyz="0"
-          izz="1e-6"
-      />
-    </inertial>
-    <collision name='collision'>
-      <origin xyz="0 0 0" rpy=" 0 0 0"/>
-      <geometry>
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